File: board/analog-eval/ph2102-analog-eval-board.kicad_pcb (KiCad board)
At the start: 2 copper layers, 38.1 x 50.8 mm, 5 parts, among them U1 LMC662, U3 REF3020, U5 LM27762

Commit message: update
Parts:
- added C1: 1u, Capacitor_SMD:C_0603_1608Metric, F.Cu at (37.8, 20.1)
- added C10: 1u, Capacitor_SMD:C_0603_1608Metric, F.Cu at (19.6, 27.4)
- added C11: 1u, Capacitor_SMD:C_0603_1608Metric, F.Cu at (24.9, 20.1)
- added C12: 100n, Capacitor_SMD:C_0603_1608Metric, F.Cu at (34.8, 39.6)
- added C13: 1u, Capacitor_SMD:C_0603_1608Metric, F.Cu at (36.6, 44.2)
- added C14: 1u, Capacitor_SMD:C_0603_1608Metric, F.Cu at (13.2, 45.0)
- added C15: 1u, Capacitor_SMD:C_0603_1608Metric, F.Cu at (17.0, 40.9)
- added C16: 4u7, Capacitor_SMD:C_0603_1608Metric, F.Cu at (18.0, 47.2)
- added C17: 10u, Capacitor_SMD:C_0603_1608Metric, F.Cu at (13.2, 46.5)
- added C18: 2u2, Capacitor_SMD:C_0603_1608Metric, F.Cu at (13.2, 42.4)
- added C19: 2u2, Capacitor_SMD:C_0603_1608Metric, F.Cu at (21.6, 45.0)
- added C2: 1u, Capacitor_SMD:C_0603_1608Metric, F.Cu at (33.5, 27.7)
- added C20: 100n, Capacitor_SMD:C_0603_1608Metric, F.Cu at (42.4, 30.0)
- added C21: 100n, Capacitor_SMD:C_0603_1608Metric, F.Cu at (37.8, 27.7)
- added C22: 100u, Capacitor_Tantalum_SMD:CP_EIA-3528-15_AVX-H, F.Cu at (12.4, 49.2)
- added C3: 100n, Capacitor_SMD:C_0603_1608Metric, F.Cu at (30.9, 25.1)
- added C4: 100n, Capacitor_SMD:C_0603_1608Metric, F.Cu at (18.3, 34.0)
- added C5: 1u, Capacitor_SMD:C_0603_1608Metric, F.Cu at (16.6, 34.0)
- added C6: 10n, Capacitor_SMD:C_0603_1608Metric, F.Cu at (28.1, 24.1)
- added C7: 1n, Capacitor_SMD:C_0603_1608Metric, F.Cu at (33.3, 36.3)
- added C8: 10u, Capacitor_SMD:C_0603_1608Metric, F.Cu at (23.9, 34.0)
- added C9: 100n, Capacitor_SMD:C_0603_1608Metric, F.Cu at (34.8, 44.2)
- added H1: M3, MountingHole:MountingHole_3.2mm_M3_Pad_Via, F.Cu at (5.08, 3.81)
- added H2: M3, MountingHole:MountingHole_3.2mm_M3_Pad_Via, F.Cu at (5.08, 59.7)
- added H3: M3, MountingHole:MountingHole_3.2mm_M3_Pad_Via, F.Cu at (40.6, 59.7)
- added H4: M3, MountingHole:MountingHole_3.2mm_M3_Pad_Via, F.Cu at (40.6, 3.81)
- added J1: CONN_PROBE, Connector_Coaxial:BNC_Amphenol_B6252HB-NPP3G-50_Horizontal, F.Cu at (17.8, 13.0)
- added J2: CONN_OUT, Connector_PinHeader_2.54mm:PinHeader_1x10_P2.54mm_Vertical, F.Cu at (11.4, 61.6)
- added J3: CONN_NTC, Connector_JST:JST_XH_S2B-XH-A-1_1x02_P2.50mm_Horizontal, F.Cu at (32.8, 7.87)
- added NT1: NetTie_2, NetTie:NetTie-2_SMD_Pad2.0mm, B.Cu at (17.3, 54.4)
- added R1: 10k/1%, Resistor_SMD:R_0603_1608Metric, F.Cu at (27.1, 29.7)
- added R10: 9.1k/1%, Resistor_SMD:R_0603_1608Metric, F.Cu at (16.5, 27.4)
- added R11: 10k, Resistor_SMD:R_0603_1608Metric, F.Cu at (27.2, 44.2)
- added R12: 10k, Resistor_SMD:R_0603_1608Metric, F.Cu at (29.7, 36.3)
- added R13: 10k, Resistor_SMD:R_0603_1608Metric, F.Cu at (23.1, 45.0)
- added R14: R_Small, Resistor_SMD:R_0603_1608Metric, F.Cu at (14.0, 40.9)
- added R15: R_Small, Resistor_SMD:R_0603_1608Metric, F.Cu at (20.8, 42.7)
- added R16: R_Small, Resistor_SMD:R_0603_1608Metric, F.Cu at (10.9, 40.9)
- added R17: R_Small, Resistor_SMD:R_0603_1608Metric, F.Cu at (20.1, 45.0)
- added R19: 10k, Resistor_SMD:R_0603_1608Metric, F.Cu at (40.6, 23.6)
- added R2: 10k/1%, Resistor_SMD:R_0603_1608Metric, F.Cu at (30.4, 29.7)
- added R21: 100R, Resistor_SMD:R_0603_1608Metric, F.Cu at (42.4, 26.9)
- added R22: 100R, Resistor_SMD:R_0603_1608Metric, F.Cu at (31.5, 36.3)
- added R23: 10k, Resistor_SMD:R_0603_1608Metric, F.Cu at (40.6, 26.9)
- added R3: 10k/1%, Resistor_SMD:R_0603_1608Metric, F.Cu at (33.7, 29.7)
- added R4: 10k/1%, Resistor_SMD:R_0603_1608Metric, F.Cu at (36.9, 29.7)
- added R5: 100k, Resistor_SMD:R_0603_1608Metric, F.Cu at (28.1, 25.9)
- added R6: 100k, Resistor_SMD:R_0603_1608Metric, F.Cu at (28.1, 22.4)
- added R8: 1M, Resistor_SMD:R_0603_1608Metric, F.Cu at (17.8, 17.9)
- added R9: 10k/1%, Resistor_SMD:R_0603_1608Metric, F.Cu at (24.9, 23.4)
- added REF**: ESD-Logo_6.6x6mm_SilkScreen, Symbol:ESD-Logo_6.6x6mm_SilkScreen, F.Cu at (40.6, 35.1)
- added REF**: WEEE-Logo_4.2x6mm_SilkScreen, Symbol:WEEE-Logo_4.2x6mm_SilkScreen, F.Cu at (40.6, 40.6)
- added REF**: KiCad-Logo2_5mm_SilkScreen, Symbol:KiCad-Logo2_5mm_SilkScreen, F.Cu at (40.6, 49.5)
- added REF**: OSHW-Logo2_7.3x6mm_SilkScreen, Symbol:OSHW-Logo2_7.3x6mm_SilkScreen, F.Cu at (41.1, 14.7)
- added TP1: TP_PGOOD, TestPoint:TestPoint_Pad_D1.0mm, F.Cu at (25.4, 40.9)
- added TP3: TP_+2V5, TestPoint:TestPoint_Pad_D1.0mm, F.Cu at (16.5, 39.1)
- added TP4: TP_-2V5, TestPoint:TestPoint_Pad_D1.0mm, F.Cu at (22.6, 40.9)
- added U2: TLV2333, Package_SO:SOIC-8_3.9x4.9mm_P1.27mm, F.Cu at (35.8, 23.9)
- added U4: MCP3201-BI/SN, Package_SO:SOIC-8_3.9x4.9mm_P1.27mm, F.Cu at (31.0, 41.9)
- R18: footprint Resistor_SMD:R_0805_2012Metric -> Resistor_SMD:R_1206_3216Metric_Pad1.30x1.75mm_HandSolder
- R7: footprint Resistor_SMD:R_0402_1005Metric -> Resistor_SMD:R_0603_1608Metric
- moved U3 73.0 mm to (21.1, 33.5), turned to 90 degrees
- moved U5 64.0 mm to (17.0, 43.7), turned to 90 degrees
- moved R18 18.7 mm to (13.6, 25.7), turned to 90 degrees
- moved R7 16.6 mm to (22.5, 25.9)
- moved U1 8.62 mm to (20.2, 22.2), turned to 180 degrees
Connections:
- U3 pad 1: +3V0 -> +2V5
- U5 pad 11: Net-(R14-Pad1) -> +2V5
- U5 pad 12: unconnected-(U5-Pad12) -> +3V3
- U5 pad 6: Net-(R15-Pad2) -> -2V5
- U5 pad 8: unconnected-(U5-Pad8) -> +3V3
Routing:
- net Net-(C6-Pad2): track 0.00 -> 23.5 mm
- net /NTC_IN: track 0.00 -> 22.9 mm
- net Net-(R10-Pad1): track 0.00 -> 18.6 mm
- net +3V3: track 0.00 -> 13.5 mm
- net GNDA: track 0.00 -> 13.3 mm, vias 0 -> 50
- net Net-(C3-Pad1): track 0.00 -> 10.9 mm
- net Net-(R13-Pad2): track 0.00 -> 10.2 mm, vias 0 -> 2
- net Net-(C6-Pad1): track 0.00 -> 8.24 mm
- net Net-(R21-Pad1): track 0.00 -> 7.70 mm
- net VREF: track 0.00 -> 6.46 mm
- net +2V5: track 3.17 -> 8.68 mm
- net Net-(R13-Pad1): track 0.00 -> 4.63 mm
- net /GUARD: track 0.00 -> 4.55 mm, vias 0 -> 15
- net -2V5: track 0.00 -> 4.53 mm
- net /VPH: track 0.00 -> 4.14 mm
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- added copper zone on F.Cu, net +2V5
- added copper zone on F.Cu, net +3V3
- added copper zone on F.Cu, net -2V5
- added copper zone on B.Cu, net /GUARD
- added copper zone on B.Cu, net GND
- added copper zone on B.Cu, net GNDA
- added copper zone on F.Cu, net GNDA
- added copper zone on F.Cu, net Net-(C16-Pad1)
- added copper zone on F.Cu, net Net-(R14-Pad2)
- added copper zone on F.Cu, net VREF
Other:
- board size 38.1 x 50.8 mm -> 43.2 x 63.5 mm
- board text added: "${COMPANY} DESIGNER: LI WEI"
- board text added: "${TITLE} PH2102_EVAL_BOARD"
- board text added: "+2.048V"
- board text added: "+3V3"
- board text added: "10k_NTC"
- board text added: "ADC_DO"
- board text added: "ADC_SCK"
- board text added: "AGND"
- board text added: "BNC 座"
- board text added: "DATE: ${ISSUE_DATE} REV: ${REVISION}"
- board text added: "GND"
- board text added: "M3*4"
- board text added: "NTC_IN"
- board text added: "NTC_OUT"
- board text added: "VPH"
- board text added: "~ADC_CS"
- board text added: "保护环焊后需清洁"
